Commit message: working spawn with wheel rotation in place forklift in gazebo with ign demo dependency

File: src/mini_task/model/forklift_robot.xacro.urdf (robot description, URDF)
Before this commit: robot forklift_robot, 6 links, 5 joints
Links:
- link base_link: geometry collision box size=2.159 1.0668 2.7432; visual mesh filename=file:///home/ahmad/ros2_ign_diffdrive/src/mini_task/model/b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
- link fork: geometry collision mesh filename=file:///home/ahmad/ros2_ign_diffdrive/src/mini_task/model/f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; visual mesh filename=file:///home/ahmad/ros2_ign_diffdrive/src/mini_task/model/f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
- link wheel_back_left: geometry collision cylinder length=0.05 radius=0.21; visual cylinder length=0.05 radius=0.21
- link wheel_back_right: geometry collision cylinder length=0.05 radius=0.21; visual cylinder length=0.05 radius=0.21
- link wheel_front_left: geometry collision cylinder length=0.05 radius=0.21; visual cylinder length=0.05 radius=0.21
- link wheel_front_right: geometry collision cylinder length=0.05 radius=0.21; visual cylinder length=0.05 radius=0.21
Joints:
- removed joint base_to_fork
- removed joint base_to_wheel_back_left
- removed joint base_to_wheel_back_right
- removed joint base_to_wheel_front_left
- removed joint base_to_wheel_front_right
- added joint fork_joint: type prismatic, parent base_link, child fork, origin xyz=2.159 0.175 0 rpy=0 0 0, axis 0 0 1, limit lower=0 upper=2 effort=100 velocity=0.1
- added joint left_wheel_steering_joint: type continuous, parent base_link, child wheel_front_left, origin xyz=1.8 0.9 0.2 rpy=1.57 0 0, axis 0 1 0
- added joint rear_left_wheel_joint: type continuous, parent base_link, child wheel_back_left, origin xyz=0.3 0.9 0.2 rpy=1.57 0 0, axis 0 0 1
- added joint rear_right_wheel_joint: type continuous, parent base_link, child wheel_back_right, origin xyz=0.3 0.1 0.2 rpy=01.57 0 0, axis 0 0 1
- added joint right_wheel_steering_joint: type continuous, parent base_link, child wheel_front_right, origin xyz=01.8 0.1 0.2 rpy=1.57 0 0, axis 0 1 0

Commit message: working motion in gazebo for forklift

File: src/mini_task/model/forklift_robot.xacro.urdf (robot description, URDF)
Before this commit: robot forklift_robot, 6 links, 5 joints
Links:
- removed link wheel_front_left
- removed link wheel_front_right
- added link chassis, mass 100; collision mesh filename=file:///home/ahmad/ros2_ign_diffdrive/src/mini_task/model/b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; visual mesh filename=file:///home/ahmad/ros2_ign_diffdrive/src/mini_task/model/b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
- added link front_left_wheel, mass 11.3; collision cylinder length=0.2 radius=0.2; visual mesh filename=file:///home/ahmad/ros2_ign_diffdrive/src/mini_task/model/w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
- added link front_right_wheel, mass 11.3; collision cylinder length=0.2 radius=0.2; visual mesh filename=file:///home/ahmad/ros2_ign_diffdrive/src/mini_task/model/w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
- added link left_wheel_steering, mass 0.1
- added link right_wheel_steering, mass 0.1
- link base_link: mass 500 -> None; geometry 
- link wheel_back_left: mass 5 -> 11.3; geometry collision cylinder length=0.2 radius=0.2; visual mesh filename=file:///home/ahmad/ros2_ign_diffdrive/src/mini_task/model/w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
- link wheel_back_right: mass 5 -> 11.3; geometry collision cylinder length=0.2 radius=0.2; visual mesh filename=file:///home/ahmad/ros2_ign_diffdrive/src/mini_task/model/w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
Joints:
- added joint base_link_to_chassis: type fixed, parent base_link, child chassis, origin xyz=0 0 0.1 rpy=0 0 0
- added joint front_left_wheel_joint: type continuous, parent left_wheel_steering, child front_left_wheel, origin xyz=0 0 0 rpy=0 0 0, axis 0 0 1
- added joint front_right_wheel_joint: type continuous, parent right_wheel_steering, child front_right_wheel, origin xyz=0 0 0 rpy=0 0 0, axis 0 0 1
- joint fork_joint: origin xyz=2.159 0.175 0 rpy=0 0 0 -> xyz=1.0795 0 0.01 rpy=0 0 0; parent base_link -> chassis
- joint left_wheel_steering_joint: child wheel_front_left -> left_wheel_steering; limit (none) -> lower=-1.57 upper=1.57 effort=1000.0 velocity=30; origin xyz=1.8 0.9 0.2 rpy=1.57 0 0 -> xyz=0.65 -0.3835 0.1 rpy=1.57 0 0; parent base_link -> chassis; type continuous -> revolute
- joint rear_left_wheel_joint: origin xyz=0.3 0.9 0.2 rpy=1.57 0 0 -> xyz=-0.7795 -0.3835 0.1 rpy=1.57 0 0; parent base_link -> chassis
- joint rear_right_wheel_joint: origin xyz=0.3 0.1 0.2 rpy=01.57 0 0 -> xyz=-0.7795 0.3835 0.1 rpy=1.57 0 0; parent base_link -> chassis
- joint right_wheel_steering_joint: child wheel_front_right -> right_wheel_steering; limit (none) -> lower=-1.57 upper=1.57 effort=1000.0 velocity=30; origin xyz=01.8 0.1 0.2 rpy=1.57 0 0 -> xyz=0.65 0.3835 0.1 rpy=1.57 0 0; parent base_link -> chassis; type continuous -> revolute

Commit message: fix paths for docker image

File: src/mini_task/model/forklift_robot.xacro.urdf (robot description, URDF)
Before this commit: robot forklift_robot, 9 links, 8 joints
Links:
- link chassis: geometry collision mesh filename=file://current_pose/workspaces/ros2-template-workspace/ros2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; visual mesh filename=file://current_pose/workspaces/ros2-template-workspace/ros2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
- link fork: geometry collision mesh filename=file://current_pose/workspaces/ros2-template-workspace/ros2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; visual mesh filename=file://current_pose/workspaces/ros2-template-workspace/ros2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
- link front_left_wheel: geometry collision cylinder length=0.2 radius=0.2; visual mesh filename=file://current_pose/workspaces/ros2-template-workspace/ros2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
- link front_right_wheel: geometry collision cylinder length=0.2 radius=0.2; visual mesh filename=file://current_pose/workspaces/ros2-template-workspace/ros2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
- link wheel_back_left: geometry collision cylinder length=0.2 radius=0.2; visual mesh filename=file://current_pose/workspaces/ros2-template-workspace/ros2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
- link wheel_back_right: geometry collision cylinder length=0.2 radius=0.2; visual mesh filename=file://current_pose/workspaces/ros2-template-workspace/ros2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

Commit message: fix wrong meshfile paths

File: src/mini_task/model/forklift_robot.xacro.urdf (robot description, URDF)
Before this commit: robot forklift_robot, 9 links, 8 joints
Links:
- link chassis: geometry collision mesh filename=file:///workspaces/ros2-template-workspace/ros2_ign_diffdri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; visual mesh filename=file:///workspaces/ros2-template-workspace/ros2_ign_diffdri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
- link fork: geometry collision mesh filename=file:///workspaces/ros2-template-workspace/ros2_ign_diffdri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; visual mesh filename=file:///workspaces/ros2-template-workspace/ros2_ign_diffdri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
- link front_left_wheel: geometry collision cylinder length=0.2 radius=0.2; visual mesh filename=file:///workspaces/ros2-template-workspace/ros2_ign_diffdri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
- link front_right_wheel: geometry collision cylinder length=0.2 radius=0.2; visual mesh filename=file:///workspaces/ros2-template-workspace/ros2_ign_diffdri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
- link wheel_back_left: geometry collision cylinder length=0.2 radius=0.2; visual mesh filename=file:///workspaces/ros2-template-workspace/ros2_ign_diffdri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
- link wheel_back_right: geometry collision cylinder length=0.2 radius=0.2; visual mesh filename=file:///workspaces/ros2-template-workspace/ros2_ign_diffdri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

Commit message: use relative path of meshfiles

File: src/mini_task/model/forklift_robot.xacro.urdf (robot description, URDF)
Before this commit: robot forklift_robot, 9 links, 8 joints
Links:
- link chassis: geometry collision mesh filename=$(find mini_task)/model/base_link.dae; visual mesh filename=$(find mini_task)/model/base_link.dae
- link fork: geometry collision mesh filename=$(find mini_task)/model/fork.dae; visual mesh filename=$(find mini_task)/model/fork.dae
- link front_left_wheel: geometry collision cylinder length=0.2 radius=0.2; visual mesh filename=$(find mini_task)/model/wheel.dae
- link front_right_wheel: geometry collision cylinder length=0.2 radius=0.2; visual mesh filename=$(find mini_task)/model/wheel.dae
- link wheel_back_left: geometry collision cylinder length=0.2 radius=0.2; visual mesh filename=$(find mini_task)/model/wheel.dae
- link wheel_back_right: geometry collision cylinder length=0.2 radius=0.2; visual mesh filename=$(find mini_task)/model/wheel.dae
