Commit message: testing fork motion

File: mini_task/model/forklift_rviz.urdf (robot description, URDF)
Before this commit: robot forklift_robot, 9 links, 8 joints
Links:
- link chassis: geometry collision mesh filename=file://$(find mini_task)/model/base_link.dae; visual mesh filename=file://$(find mini_task)/model/base_link.dae
- link fork: mass 100 -> 10; geometry collision mesh filename=file://$(find mini_task)/model/fork.dae; visual mesh filename=file://$(find mini_task)/model/fork.dae
- link front_left_wheel: geometry collision cylinder length=0.2 radius=0.2; visual mesh filename=file://$(find mini_task)/model/wheel.dae
- link front_right_wheel: geometry collision cylinder length=0.2 radius=0.2; visual mesh filename=file://$(find mini_task)/model/wheel.dae
- link wheel_back_left: geometry collision cylinder length=0.2 radius=0.2; visual mesh filename=file://$(find mini_task)/model/wheel.dae
- link wheel_back_right: geometry collision cylinder length=0.2 radius=0.2; visual mesh filename=file://$(find mini_task)/model/wheel.dae
