Commit message: working fork motion

File: model/forklift_robot.urdf.xacro (robot description, xacro)
@@ -31,5 +31,5 @@
   </link>
   <joint name="base_link_to_chassis" type="fixed">
-    <origin rpy="0 0 0" xyz="0 0 0.1" />
+    <origin rpy="0 0 0" xyz="0 0 0" />
     <parent link="base_link" />
     <child link="chassis" />
@@ -50,5 +50,5 @@
     </collision>
     <inertial>
-      <mass value="100" />
+      <mass value="10" />
       <inertia ixx="0.2" ixy="0" ixz="0" iyy="0.3" iyz="0" izz="0.4" />
     </inertial>
@@ -133,74 +133,9 @@
     <dynamics damping="0.2" />
   </joint>
-  <!--
-  <link name="wheel_front_left">
-    <visual>
-      <geometry>
-        <mesh filename="$(find ros2_ign_p2p_controllers)/model/wheel.dae" />
-      </geometry>
-      <material name="Black" />
-    </visual>
-    <collision>
-      <geometry>
-        <cylinder radius="0.2" length="0.2" />
-      </geometry>
-    </collision>
-    <inertial>
-      <mass value="5.2" />
-      <inertia ixx="0.0001" ixy="0" ixz="0" iyy="0.0001" iyz="0" izz="0.0001" />
-    </inertial>
-    <surface>
-      <friction>
-        <ode>
-          <mu>1.0</mu>
-          <mu2>1.0</mu2>
-        </ode>
-      </friction>
-    </surface>
-  </link>
-  <joint name="left_wheel_steering_joint" type="continuous">
-    <origin xyz="0.65 -0.3835 0.1" rpy="1.57 0 0" />
-    <parent link="chassis" />
-    <child link="wheel_front_left" />
-    <axis xyz="0 1 0" />
-    <dynamics damping="0.2" />
-  </joint>
-  <link name="wheel_front_right">
-    <visual>
-      <geometry>
-        <mesh filename="$(find ros2_ign_p2p_controllers)/model/wheel.dae" />
-      </geometry>
-      <material name="Black" />
-    </visual>
-    <collision>
-      <geometry>
-        <cylinder radius="0.2" length="0.2" />
-      </geometry>
-    </collision>
-    <inertial>
-      <mass value="5.2" />
-      <inertia ixx="0.0001" ixy="0" ixz="0" iyy="0.0001" iyz="0" izz="0.0001" />
-    </inertial>
-    <surface>
-      <friction>
-        <ode>
-          <mu>1.0</mu>
-          <mu2>1.0</mu2>
-        </ode>
-      </friction>
-    </surface>
-  </link>
-  <joint name="right_wheel_steering_joint" type="continuous">
-    <origin xyz="0.65 0.3835 0.1" rpy="1.57 0 0" />
-    <parent link="chassis" />
-    <child link="wheel_front_right" />
-    <axis xyz="0 1 0" />
-    <dynamics damping="0.2" />
-  </joint> -->
   <!-- left steer Link -->
   <link name="left_wheel_steering">
     <inertial>
       <mass value="0.1" />
-      <inertia ixx="0" ixy="0.0" ixz="0.0" iyy="0.0" iyz="0.0" izz="0.0" />
+      <inertia ixx="0.002" ixy="0.0" ixz="0.0" iyy="0.002" iyz="0.0" izz="0.002" />
     </inertial>
   </link>
@@ -217,5 +152,5 @@
     <inertial>
       <mass value="0.1" />
-      <inertia ixx="0" ixy="0.0" ixz="0.0" iyy="0.0" iyz="0.0" izz="0.0" />
+      <inertia ixx="0.002" ixy="0.0" ixz="0.0" iyy="0.002" iyz="0.0" izz="0.002" />
     </inertial>
   </link>
@@ -301,5 +236,5 @@
     </joint>
     <joint name="fork_joint">
-      <command_interface name="position"/>
+      <command_interface name="position" />
       <state_interface name="position">
         <param name="initial_value">0.2</param>

File: model/forklift_rviz.urdf (robot description, URDF)
Before this commit: robot forklift_robot, 9 links, 8 joints
Links:
- link chassis: geometry collision mesh filename=package://ros2_ign_p2p_controllers/model/base_link.dae; visual mesh filename=package://ros2_ign_p2p_controllers/model/base_link.dae
- link fork: geometry collision mesh filename=package://ros2_ign_p2p_controllers/model/fork.dae; visual mesh filename=package://ros2_ign_p2p_controllers/model/fork.dae
- link front_left_wheel: geometry collision cylinder length=0.2 radius=0.2; visual mesh filename=package://ros2_ign_p2p_controllers/model/wheel.dae
- link front_right_wheel: geometry collision cylinder length=0.2 radius=0.2; visual mesh filename=package://ros2_ign_p2p_controllers/model/wheel.dae
- link wheel_back_left: geometry collision cylinder length=0.2 radius=0.2; visual mesh filename=package://ros2_ign_p2p_controllers/model/wheel.dae
- link wheel_back_right: geometry collision cylinder length=0.2 radius=0.2; visual mesh filename=package://ros2_ign_p2p_controllers/model/wheel.dae
Joints:
- joint base_link_to_chassis: origin xyz=0 0 0.1 rpy=0 0 0 -> xyz=0 0 0 rpy=0 0 0

Commit message: update palette in gazebo

File: model/forklift_robot.urdf.xacro (robot description, xacro)
@@ -31,5 +31,5 @@
   </link>
   <joint name="base_link_to_chassis" type="fixed">
-    <origin rpy="0 0 0" xyz="0 0 0" />
+    <origin rpy="0 0 0" xyz="0 0 0.05" />
     <parent link="base_link" />
     <child link="chassis" />
@@ -52,35 +52,4 @@
       <mass value="10" />
       <inertia ixx="0.2" ixy="0" ixz="0" iyy="0.3" iyz="0" izz="0.4" />
-    </inertial>
-  </link>
-  <joint name="fork_joint" type="prismatic">
-    <origin rpy="0 0 0" xyz="1.0795 0 0.01" />
-    <parent link="chassis" />
-    <child link="fork" />
-    <limit
-      lower="0"
-      upper="2"
-      velocity="0.1"
-      effort="100"
-    />
-    <axis xyz="0 0 1" />
-    <dynamics damping="0.2" />
-  </joint>
-  <link name="wheel_back_left">
-    <visual>
-      <!-- <origin xyz="-0.2 0.2 -0.1" rpy="1.5707 0 0" /> -->
-      <geometry>
-        <mesh filename="$(find ros2_ign_p2p_controllers)/model/wheel.dae" />
-      </geometry>
-      <material name="Black" />
-    </visual>
-    <collision>
-      <geometry>
-        <cylinder radius="0.2" length="0.2" />
-      </geometry>
-    </collision>
-    <inertial>
-      <mass value="11.3" />
-      <inertia ixx="0.26" ixy="0.0" ixz="0.0" iyy="0.26" iyz="0.0" izz="0.51" />
     </inertial>
     <surface>
@@ -93,12 +62,18 @@
     </surface>
   </link>
-  <joint name="rear_left_wheel_joint" type="continuous">
-    <origin xyz="-0.7795 -0.3835 0.1" rpy="1.57 0 0" />
-    <parent link="chassis" />
-    <child link="wheel_back_left" />
-    <axis xyz="0 0 1" />
-    <dynamics damping="0.2" />
-  </joint>
-  <link name="wheel_back_right">
+  <joint name="fork_joint" type="prismatic">
+    <origin rpy="0 0 0" xyz="1.0795 0 0.002" />
+    <parent link="chassis" />
+    <child link="fork" />
+    <limit
+      lower="0"
+      upper="2"
+      velocity="0.1"
+      effort="100"
+    />
+    <axis xyz="0 0 1" />
+    <dynamics damping="0.2" />
+  </joint>
+  <link name="wheel_back_left">
     <visual>
       <!-- <origin xyz="-0.2 0.2 -0.1" rpy="1.5707 0 0" /> -->
@@ -126,4 +101,37 @@
     </surface>
   </link>
+  <joint name="rear_left_wheel_joint" type="continuous">
+    <origin xyz="-0.7795 -0.3835 0.1" rpy="1.57 0 0" />
+    <parent link="chassis" />
+    <child link="wheel_back_left" />
+    <axis xyz="0 0 1" />
+    <dynamics damping="0.2" />
+  </joint>
+  <link name="wheel_back_right">
+    <visual>
+      <!-- <origin xyz="-0.2 0.2 -0.1" rpy="1.5707 0 0" /> -->
+      <geometry>
+        <mesh filename="$(find ros2_ign_p2p_controllers)/model/wheel.dae" />
+      </geometry>
+      <material name="Black" />
+    </visual>
+    <collision>
+      <geometry>
+        <cylinder radius="0.2" length="0.2" />
+      </geometry>
+    </collision>
+    <inertial>
+      <mass value="11.3" />
+      <inertia ixx="0.26" ixy="0.0" ixz="0.0" iyy="0.26" iyz="0.0" izz="0.51" />
+    </inertial>
+    <surface>
+      <friction>
+        <ode>
+          <mu>1.0</mu>  <!-- Friction coefficient -->
+          <mu2>1.0</mu2>
+        </ode>
+      </friction>
+    </surface>
+  </link>
   <joint name="rear_right_wheel_joint" type="continuous">
     <origin xyz="-0.7795 0.3835 0.1" rpy="1.57 0 0" />
